File: Practica2/Microcontrolador.kicad_sch (KiCad schematic)
At the start: 8 parts, among them J1 Conn_01x04, U2 ATtiny3216-S

Commit message: Practica3
Avance de la P3
Parts:
- removed J1: Conn_01x04, Connector_PinHeader_2.54mm:PinHeader_1x04_P2.54mm_Vertical, symbol Connector_Generic:Conn_01x04
- added C6: 100nF, Capacitor_SMD:C_0603_1608Metric, symbol Device:C
Connections:
- net 3V3: now also C6.1
- net GND: now also C6.2
Changed lines of the file:
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@@
 	(paper "A4")
+	(junction
+		(at 135.89 143.51)
+		(diameter 0)
+		(color 0 0 0 0)
+	)
 	(junction
 		(at 209.55 127)
@@
 		(color 0 0 0 0)
 	)
+	(junction
+		(at 135.89 88.9)
+		(diameter 0)
+		(color 0 0 0 0)
+	)
 	(no_connect
 		(at 151.13 115.57)
@@
 	(wire
 		(pts
-			(xy 241.3 118.11) (xy 251.46 118.11)
-		)
-		(stroke
-			(width 0)
-			(type default)
-		)
-	)
-	(wire
-		(pts
-			(xy 135.89 140.97) (xy 135.89 148.59)
+			(xy 135.89 140.97) (xy 135.89 143.51)
 		)
 		(stroke
@@
 	(wire
 		(pts
-			(xy 251.46 115.57) (xy 241.3 115.57)
-		)
-		(stroke
-			(width 0)
-			(type default)
-		)
-	)
-	(wire
-		(pts
 			(xy 187.96 127) (xy 213.36 127)
 		)
@@
 	(wire
 		(pts
+			(xy 135.89 88.9) (xy 135.89 95.25)
+		)
+		(stroke
+			(width 0)
+			(type default)
+		)
+	)
+	(wire
+		(pts
+			(xy 135.89 143.51) (xy 135.89 148.59)
+		)
+		(stroke
+			(width 0)
+			(type default)
+		)
+	)
+	(wire
+		(pts
+			(xy 101.6 100.33) (xy 101.6 88.9)
+		)
+		(stroke
+			(width 0)
+			(type default)
+		)
+	)
+	(wire
+		(pts
 			(xy 151.13 105.41) (xy 186.69 105.41)
 		)
@@
 	(wire
 		(pts
-			(xy 135.89 78.74) (xy 135.89 95.25)
+			(xy 135.89 78.74) (xy 135.89 88.9)
+		)
+		(stroke
+			(width 0)
+			(type default)
+		)
+	)
+	(wire
+		(pts
+			(xy 101.6 143.51) (xy 135.89 143.51)
 		)
 		(stroke
@@
 	(wire
 		(pts
-			(xy 251.46 120.65) (xy 241.3 120.65)
-		)
-		(stroke
-			(width 0)
-			(type default)
-		)
-	)
-	(wire
-		(pts
 			(xy 187.96 107.95) (xy 187.96 127)
 		)
@@
 	(wire
 		(pts
+			(xy 101.6 107.95) (xy 101.6 143.51)
+		)
+		(stroke
+			(width 0)
+			(type default)
+		)
+	)
+	(wire
+		(pts
 			(xy 234.95 80.01) (xy 234.95 82.55)
 		)
@@
 	(wire
 		(pts
-			(xy 241.3 113.03) (xy 251.46 113.03)
+			(xy 101.6 88.9) (xy 135.89 88.9)
 		)
 		(stroke
@@
 	(label "3V3"
 		(at 135.89 86.36 0)
-		(effects
-			(font
-				(size 1.27 1.27)
-			)
-			(justify left bottom)
-		)
-	)
-	(label "IN3"
-		(at 241.3 120.65 0)
-		(effects
-			(font
-				(size 1.27 1.27)
-			)
-			(justify left bottom)
-		)
-	)
-	(label "3V3"
-		(at 241.3 113.03 0)
-		(effects
-			(font
-				(size 1.27 1.27)
-			)
-			(justify left bottom)
-		)
-	)
-	(label "IN2"
-		(at 241.3 118.11 0)
-		(effects
-			(font
-				(size 1.27 1.27)
-			)
-			(justify left bottom)
-		)
-	)
-	(label "IN1"
-		(at 241.3 115.57 0)
 		(effects
 			(font
@@
 			)
 			(justify left)
-		)
-	)
-	(symbol
-		(lib_id "Connector_Generic:Conn_01x04")
-		(at 256.54 115.57 0)
-		(unit 1)
-		(body_style 1)
-		(exclude_from_sim no)
-		(in_bom yes)
-		(on_board yes)
-		(in_pos_files yes)
-		(dnp no)
-		(fields_autoplaced yes)
-		(property "Reference" "J1"
-			(at 259.08 115.5699 0)
-			(show_name no)
-			(do_not_autoplace no)
-			(effects
-				(font
-					(size 1.27 1.27)
-				)
-				(justify left)
-			)
-		)
-		(property "Value" "Conn_01x04"
-			(at 259.08 118.1099 0)
-			(show_name no)
-			(do_not_autoplace no)
-			(effects
-				(font
-					(size 1.27 1.27)
-				)
-				(justify left)
-			)
-		)
-		(property "Footprint" "Connector_PinHeader_2.54mm:PinHeader_1x04_P2.54mm_Vertical"
-			(at 256.54 115.57 0)
-			(hide yes)
-			(show_name no)
-			(do_not_autoplace no)
-			(effects
-				(font
-					(size 1.27 1.27)
-				)
-			)
-		)
-		(property "Datasheet" ""
-			(at 256.54 115.57 0)
-			(hide yes)
-			(show_name no)
-			(do_not_autoplace no)
-			(effects
-				(font
-					(size 1.27 1.27)
-				)
-			)
-		)
-		(property "Description" "Generic connector, single row, 01x04, script generated (kicad-library-utils/schlib/autogen/connector/)"
-			(at 256.54 115.57 0)
-			(hide yes)
-			(show_name no)
-			(do_not_autoplace no)
-			(effects
-				(font
-					(size 1.27 1.27)
-				)
-			)
-		)
-		(property "MPN" "61300411121"
-			(at 256.54 115.57 0)
-			(hide yes)
-			(show_name no)
-			(do_not_autoplace no)
-			(effects
-				(font
-					(size 1.27 1.27)
-				)
-			)
-		)
-		(pin "1"
-		)
-		(pin "3"
-		)
-		(pin "2"
-		)
-		(pin "4"
-		)
-		(instances
-			(project "Practica2"
-				(path "/a80ac9b4-6a18-46be-9769-32271ad0f9b9/0cb31d1a-5542-40d6-b496-d28e7e3f6c25"
-					(reference "J1")
-					(unit 1)
-				)
-			)
 		)
 	)
@@
 					(unit 1)
 				)
+			)
+		)
+	)
+	(symbol
+		(lib_id "Device:C")
+		(at 101.6 104.14 0)
+		(unit 1)
+		(body_style 1)
+		(exclude_from_sim no)
+		(in_bom yes)
+		(on_board yes)
+		(in_pos_files yes)
+		(dnp no)
+		(fields_autoplaced yes)
+		(property "Reference" "C6"
+			(at 105.41 102.8699 0)
+			(show_name no)
+			(do_not_autoplace no)
+			(effects
+				(font
+					(size 1.27 1.27)
+				)
+				(justify left)
+			)
+		)
+		(property "Value" "100nF"
+			(at 105.41 105.4099 0)
+			(show_name no)
+			(do_not_autoplace no)
+			(effects
+				(font
+					(size 1.27 1.27)
+				)
+				(justify left)
+			)
+		)
+		(property "Footprint" "Capacitor_SMD:C_0603_1608Metric"
+			(at 102.5652 107.95 0)
+			(hide yes)
+			(show_name no)
+			(do_not_autoplace no)
+			(effects
+				(font
+					(size 1.27 1.27)
+				)
+			)
+		)
+		(property "Datasheet" ""
+			(at 101.6 104.14 0)
+			(hide yes)
+			(show_name no)
+			(do_not_autoplace no)
+			(effects
+				(font
+					(size 1.27 1.27)
+				)
+			)
+		)
+		(property "Description" "Unpolarized capacitor"
+			(at 101.6 104.14 0)
+			(hide yes)
+			(show_name no)
+			(do_not_autoplace no)
+			(effects
+				(font
+					(size 1.27 1.27)
+				)
+			)
+		)
+		(pin "2"
+		)
+		(pin "1"
+		)
+		(instances
+			(project "Practica2"
+				(path "/a80ac9b4-6a18-46be-9769-32271ad0f9b9/0cb31d1a-5542-40d6-b496-d28e7e3f6c25"
+					(reference "C6")
+					(unit 1)
+				)

Commit message: Actualización P4
Parts:
- added R4, R6: 4,7k, Resistor_SMD:R_0603_1608Metric, symbol Device:R
- added R5: 4.7k, Resistor_SMD:R_0603_1608Metric, symbol Device:R
- added U3: LM75B, Package_SO:VSSOP-8_2.3x2mm_P0.5mm, symbol Sensor_Temperature:LM75B
- added U4: BME280, Package_LGA:Bosch_LGA-8_2.5x2.5mm_P0.65mm_ClockwisePinNumbering, symbol Sensor:BME280
- added U5: DS18B20, Package_TO_SOT_THT:TO-92_Inline, symbol Sensor_Temperature:DS18B20
Connections:
- net 3V3: now also R4.2, R5.2, R6.1, U3.8 (+Vs), U4.6 (VDDIO), U4.8 (VDD), U5.3 (V_{DD})
- net GND: now also U3.4 (GND), U3.5 (A2), U3.6 (A1), U3.7 (A0), U4.1 (GND), U4.7 (GND), U5.1 (GND)
- net SDA: now reaches U2.10 (PB1)
- net SDA: now also R4.1, U3.1 (SDA)
- net SCL: now reaches U2.11 (PB0)
- net SCL: now also R5.1, U3.2 (SCL)
- net SCK: now reaches U2.12 (PC0)
- net SCK: now also U4.4 (SCK)
- net MISO: now reaches U2.13 (PC1)
- net MISO: now also U4.5 (SDO)
- net MOSI: now reaches U2.14 (PC2)
- net MOSI: now also U4.3 (SDI)
- net CS: now reaches U2.15 (PC3)
- net CS: now also U4.2 (CSB)
- net ONEWIRE: now reaches U2.9 (PB2)
- net ONEWIRE: now also R6.2, U5.2 (DQ)
- no-connect marks 15 -> 9
