File: Practica2/Practica2.kicad_pcb (KiCad board)
At the start: 2 copper layers, 36.5 x 26 mm, 13 parts, among them J2 Conn_01x03, J3 Conn_01x02, U1 LD1117S33TR_SOT223, U2 ATtiny3216-S

Commit message: Practica 3- PCB terminada
Parts:
- moved C5 7.73 mm to (137.0, 91.8)
- moved C4 4.17 mm to (137.0, 94.8)
- moved R1 1.68 mm to (140.2, 97.0)
- moved R3 1.68 mm to (140.2, 91.0)
- moved R2 1.35 mm to (140.2, 94.0)
- moved C3 1.00 mm to (137.0, 97.8)
- turned C1 to -90 degrees
Routing:
- net /Microcontrolador/3V3: track 0.00 -> 32.9 mm
- net GND: track 0.00 -> 12.1 mm, vias 0 -> 8
- net /Alimentación/VI: track 3.69 -> 8.43 mm
- net Net-(U2-PA3): track 9.91 -> 11.7 mm
- net Net-(U2-PA1): track 9.69 -> 11.5 mm
- net Net-(U2-PA2): track 9.66 -> 11.0 mm
- net /Microcontrolador/IN2: track 4.37 -> 3.03 mm
- net /Microcontrolador/IN1: track 4.54 -> 3.22 mm
- net /Microcontrolador/IN3: track 4.60 -> 4.02 mm
- added copper zone on B.Cu, net GND

Commit message: Actualización P4
Parts:
- added R4: 4,7k, Resistor_SMD:R_0603_1608Metric, F.Cu at (132.2, 109.5)
- added R5: 4.7k, Resistor_SMD:R_0603_1608Metric, F.Cu at (132.2, 114.0)
- added R6: 4,7k, Resistor_SMD:R_0603_1608Metric, F.Cu at (112.7, 105.5)
- added U3: LM75B, Package_SO:VSSOP-8_2.3x2mm_P0.5mm, F.Cu at (121.0, 111.7)
- added U4: BME280, Package_LGA:Bosch_LGA-8_2.5x2.5mm_P0.65mm_ClockwisePinNumbering, F.Cu at (138.5, 103.0)
- added U5: DS18B20, Package_TO_SOT_THT:TO-92_Inline, F.Cu at (111.7, 100.9)
Connections:
- U2 pad 10: unconnected-(U2-PB1-Pad10) -> /Microcontrolador/SDA
- U2 pad 11: unconnected-(U2-PB0-Pad11) -> /Microcontrolador/SCL
- U2 pad 12: unconnected-(U2-PC0-Pad12) -> /Microcontrolador/SCK
- U2 pad 13: unconnected-(U2-PC1-Pad13) -> /Microcontrolador/MISO
- U2 pad 14: unconnected-(U2-PC2-Pad14) -> /Microcontrolador/MOSI
- U2 pad 15: unconnected-(U2-PC3-Pad15) -> /Microcontrolador/CS
- U2 pad 9: unconnected-(U2-PB2-Pad9) -> /Microcontrolador/ONEWIRE
Routing:
- net /Microcontrolador/SDA: track 0.00 -> 1.25 mm
Other:
- board outline removed
- copper layers 2 -> 4
